File: Diversity2.brd (EAGLE design)
At the start: 100 x 80 mm, 71 parts, among them IC1 LM1881, IC2 LM1881, IC3 7805TV, IC4 NE5532N, IC5 LM1881, IC6 LM1881, IC7 MEGA16-P, IC9 4052N, Q2 16MHz, U1 AD812ANZ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

Commit message: noch etwas gefummelt.
Parts:
- removed S1: (no value), switch-omron:B3F-10XX
- added SV1: (no value), con-harting-ml:ML16
- moved R14 20.5 mm to (45.7, 1.27), turned to 0 degrees
- moved C18 10.2 mm to (19.1, 38.1)
- moved C22 2.54 mm to (43.2, 6.35)
- moved C23 2.54 mm to (61.0, 6.35)
- moved Q2 2.54 mm to (52.1, 6.35)
- moved IC7 2.54 mm to (47.0, 19.1)
- moved C1 1.27 mm to (52.1, 47.0)
- moved C15 1.27 mm to (36.8, 47.0)
- moved C16 1.27 mm to (24.1, 47.0)
- moved C2 1.27 mm to (64.8, 47.0)
- moved IC1 1.27 mm to (54.6, 38.1)
- moved IC2 1.27 mm to (67.3, 38.1)
- moved IC5 1.27 mm to (39.4, 38.1)
- moved IC6 1.27 mm to (26.7, 38.1)
- moved C17 1.27 mm to (36.8, 30.5)
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Connections:
- new net N$24: IC7.1, SV1.15
- new net N$38: IC7.2, SV1.13
- new net N$50: IC7.3, SV1.11
- new net N$51: IC7.4, SV1.9
- new net N$52: IC7.5, SV1.7
- new net N$53: IC7.6, SV1.5
- new net N$54: IC7.7, SV1.3
- new net N$55: IC7.8, SV1.1
- net GND: now also SV1.2; no longer S1.3
- net N$33: now also SV1.4; no longer S1.2
Routing:
- net +5V: track 192.2 -> 159.7 mm
- net GND: track 515.1 -> 531.6 mm
- net N$53: track 0.00 -> 7.18 mm
- net N$52: track 0.00 -> 7.18 mm
- net N$51: track 0.00 -> 7.18 mm
- net N$50: track 0.00 -> 7.18 mm
- net N$55: track 0.00 -> 7.18 mm
- net N$54: track 0.00 -> 7.18 mm
- net N$38: track 0.00 -> 7.18 mm
- net N$24: track 0.00 -> 7.18 mm
- net N$33: track 17.7 -> 21.7 mm
- net N$23: track 88.9 -> 86.0 mm
- net N$22: track 3.81 -> 6.66 mm
- net N$21: track 77.7 -> 75.1 mm
- net N$15: track 40.0 -> 38.0 mm
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