File: Diversity2.brd (EAGLE design)
At the start: 100 x 100 mm, 73 parts, among them IC1 LM1881, IC2 LM1881, IC3 7805TV, IC4 NE5532N, IC5 LM1881, IC6 LM1881, IC7 MEGA16-P, IC9 4052N, Q2 16MHz, U1 AD812ANZ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

Commit message: asdf
Parts:
- added C31: 100uF, capacitor-wima:C2.5-2
- added C32: 10nF, capacitor-wima:C2.5-2
- added D2: 1N4004, diode:DO41-10
- added D3: (no value), diode:CB417-15
- added J2: (no value), con-jack:SPC4077
- added U2: LM2675N-5.0, NSC_By_element14_Batch_1.1:DIP254P762X508-8
Connections:
- new net N$62: C32.2, U2.1
- new net N$63: C31.2, D2.C, U2.7
- new net N$64: C32.1, D3.C, U2.8
- net +12V: now also D2.A, J2.3
- net GND: now also C31.1, D3.A, J2.1, J2.2, U2.6
Changed lines of the file:
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@@
 <?xml version="1.0" encoding="utf-8"?>
 <!DOCTYPE eagle SYSTEM "eagle.dtd">
-<eagle version="6.4">
+<eagle version="6.5.0">
 <drawing>
 <settings>
@@
 <attribute name="OC_FARNELL" value="unknown" x="1.27" y="-13.97" size="1.778" layer="27" display="off"/>
 </element>
+<element name="J2" library="con-jack" package="SPC4077" value="" x="-10.16" y="-24.13">
+<attribute name="OC_NEWARK" value="unknown" x="-10.16" y="-24.13" size="1.778" layer="27" display="off"/>
+<attribute name="MPN" value="" x="-10.16" y="-24.13" size="1.778" layer="27" display="off"/>
+<attribute name="MF" value="" x="-10.16" y="-24.13" size="1.778" layer="27" display="off"/>
+<attribute name="OC_FARNELL" value="unknown" x="-10.16" y="-24.13" size="1.778" layer="27" display="off"/>
+</element>
+<element name="D2" library="diode" package="DO41-10" value="1N4004" x="-15.24" y="-39.37"/>
+<element name="C31" library="capacitor-wima" package="C2.5-2" value="100uF" x="-19.05" y="-46.99"/>
+<element name="U2" library="NSC_By_element14_Batch_1.1" package="DIP254P762X508-8" value="LM2675N-5.0" x="-25.4" y="-54.61">
+<attribute name="PACKAGE" value="8-DIP" x="-25.4" y="-54.61" size="1.778" layer="27" display="off"/>
+<attribute name="OC_NEWARK" value="41K4149" x="-25.4" y="-54.61" size="1.778" layer="27" display="off"/>
+<attribute name="MPN" value="LM2675N-5.0" x="-25.4" y="-54.61" size="1.778" layer="27" display="off"/>
+<attribute name="SUPPLIER" value="NationalSemiconductor" x="-25.4" y="-54.61" size="1.778" layer="27" display="off"/>
+<attribute name="OC_FARNELL" value="9489819" x="-25.4" y="-54.61" size="1.778" layer="27" display="off"/>
+</element>
+<element name="C32" library="capacitor-wima" package="C2.5-2" value="10nF" x="-31.75" y="-63.5"/>
+<element name="D3" library="diode" package="CB417-15" value="" x="-24.13" y="-71.12"/>
 </elements>
 <signals>
@@
 <wire x1="55.88" y1="19.05" x2="55.88" y2="12.7" width="0.254" layer="1"/>
 <wire x1="55.88" y1="19.05" x2="56.2" y2="19.05" width="0.254" layer="1"/>
+<contactref element="J2" pad="1"/>
+<contactref element="J2" pad="2"/>
+<contactref element="C31" pad="1"/>
+<contactref element="U2" pad="6"/>
+<contactref element="D3" pad="A"/>
+<wire x1="-25.4" y1="-52.07" x2="-16.51" y2="-71.12" width="0" layer="19" extent="1-1"/>
+<wire x1="-20.32" y1="-46.99" x2="-25.4" y2="-52.07" width="0" layer="19" extent="1-1"/>
+<wire x1="-10.16" y1="-28.93" x2="-20.32" y2="-46.99" width="0" layer="19" extent="1-1"/>
+<wire x1="-13.16" y1="-24.13" x2="-10.16" y2="-28.93" width="0" layer="19" extent="1-1"/>
+<wire x1="7.06" y1="32.59" x2="-13.16" y2="-24.13" width="0" layer="19" extent="1-1"/>
 </signal>
 <signal name="+12V">
@@
 <wire x1="82.55" y1="27.94" x2="67.31" y2="43.18" width="0.254" layer="1"/>
 <wire x1="59.69" y1="74.93" x2="59.69" y2="74.61" width="0.254" layer="1"/>
+<contactref element="J2" pad="3"/>
+<contactref element="D2" pad="A"/>
+<wire x1="-7.16" y1="-24.13" x2="82.55" y2="7.3" width="0" layer="19" extent="1-1"/>
+<wire x1="-10.16" y1="-39.37" x2="-7.16" y2="-24.13" width="0" layer="19" extent="1-1"/>
 </signal>
 <signal name="N$5">
@@
 <wire x1="27.94" y1="1.27" x2="27.94" y2="8.57" width="0.4064" layer="1"/>
 </signal>
+<signal name="N$63">
+<contactref element="D2" pad="C"/>
+<contactref element="C31" pad="2"/>
+<contactref element="U2" pad="7"/>
+<wire x1="-17.78" y1="-46.99" x2="-25.4" y2="-49.53" width="0" layer="19" extent="1-1"/>
+<wire x1="-20.32" y1="-39.37" x2="-17.78" y2="-46.99" width="0" layer="19" extent="1-1"/>
+</signal>
+<signal name="N$62">
+<contactref element="U2" pad="1"/>
+<contactref element="C32" pad="2"/>
+<wire x1="-33.02" y1="-46.99" x2="-30.48" y2="-63.5" width="0" layer="19" extent="1-1"/>
+</signal>
+<signal name="N$64">
+<contactref element="U2" pad="8"/>
+<contactref element="C32" pad="1"/>
+<contactref element="D3" pad="C"/>
+<wire x1="-33.02" y1="-63.5" x2="-31.75" y2="-71.12" width="0" layer="19" extent="1-1"/>
+<wire x1="-25.4" y1="-46.99" x2="-33.02" y2="-63.5" width="0" layer="19" extent="1-1"/>
+</signal>
 </signals>
