File: Diversity2.sch (EAGLE design)
At the start: 71 parts, among them IC1 LM1881, IC2 LM1881, IC3 7805TV, IC4 NE5532N, IC5 LM1881, IC6 LM1881, IC7 MEGA16-P, IC9 4052N, Q2 16MHz, U1 AD812ANZ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

Commit message: so ist das
Parts:
- added SV2: (no value), con-harting-ml:ML6L
- added X4: 22-23-2031, con-molex:22-23-2031
Connections:
- new net N$56: IC7.(RXD)PD0, X4-1.S
- new net N$57: IC7.(TXD)PD1, X4-2.S
- new net N$58: IC7.(INT1)PD3, SV1.6
- new net N$59: IC7.(OC1B)PD4, SV1.8
- new net N$60: IC7.(OC1A)PD5, SV1.10
- new net N$61: IC7.(ICP)PD6, SV1.12
- net +12V: no longer IC1.VCC, IC2.VCC, IC4P.V+, IC5.VCC, IC6.VCC
- net +5V: now also IC1.VCC, IC2.VCC, IC4P.V+, IC5.VCC, IC6.VCC
- net GND: now also IC7.GND@1, SV1.1, X4-3.S; no longer SV1.2
- net N$33: now also SV1.2; no longer SV1.4
- net N$55: now also IC7.(INT0)PD2, SV1.4; no longer IC7.(SCK)PB7, SV1.1
Other:
- moved on the sheet: C21, C22, C23, IC7, Q2, R14, SV1

Commit message: asdf
Parts:
- added C31: 100uF, capacitor-wima:C2.5/2
- added C32: 10nF, capacitor-wima:C2.5/2
- added D2: 1N4004, diode:1N4004
- added D3: (no value), diode:SCHOTTKY-DIODECB417-15
- added J2: (no value), con-jack:JACK-PLUG0
- added U2: LM2675N-5.0, NSC_By_element14_Batch_1.1:LM2675N-5.0
Connections:
- new net N$62: C32.2, U2.BOOST
- new net N$63: C31.2, D2.C, U2.VIN
- new net N$64: C32.1, D3.C, U2.SW
- net +12V: now also D2.A, J2.3
- net GND: now also C31.1, D3.A, J2.1, J2.2, U2.GND
Other:
- moved on the sheet: C12, C13, C5, C6, D1, IC3, J1, R15, R16
