File: TMP/Diversity2.brd (EAGLE design)
At the start: 100 x 80 mm, 71 parts, among them IC1 LM1881, IC2 LM1881, IC3 7805TV, IC4 NE5532N, IC5 LM1881, IC6 LM1881, IC7 MEGA16-P, IC9 4052N, Q2 16MHz, U1 AD812ANZ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

Commit message: jaja
Parts:
- moved C26 92.8 mm to (85.1, 17.8)
- moved R14 83.0 mm to (66.0, 76.2), turned to 0 degrees
- moved C12 73.3 mm to (22.9, 59.7)
- moved C21 71.4 mm to (36.8, 63.5), turned to 0 degrees
- moved R3 70.0 mm to (36.8, 3.81), turned to 180 degrees
- moved C5 67.1 mm to (21.6, 52.1), turned to 0 degrees
- moved IC3 63.5 mm to (29.2, 55.9)
- moved C13 63.0 mm to (40.6, 64.8), turned to 0 degrees
- moved C6 61.7 mm to (38.1, 55.9), turned to 0 degrees
- moved C9 59.1 mm to (15.2, 8.89), turned to 0 degrees
- moved J1 55.0 mm to (77.5, 62.2), turned to 0 degrees
- moved C7 53.4 mm to (26.7, 5.08), turned to 90 degrees
- moved U1 50.9 mm to (27.9, 77.5)
- moved C10 50.4 mm to (15.2, 24.1), turned to 0 degrees
- moved C4 50.3 mm to (15.2, 63.5)
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Routing:
- net N$12: track 4.86 -> 156.7 mm
- net N$6: track 3.81 -> 109.1 mm
- net N$33: track 17.7 -> 122.2 mm
- net N$37: track 11.0 -> 104.0 mm
- net N$5: track 3.81 -> 89.5 mm
- net N$25: track 4.86 -> 89.9 mm, vias 0 -> 1
- net N$4: track 3.81 -> 85.7 mm, vias 0 -> 1
- net N$23: track 88.9 -> 7.70 mm
- net N$16: track 4.86 -> 74.3 mm, vias 0 -> 1
- net N$47: track 25.7 -> 83.7 mm, vias 0 -> 1
- net N$48: track 6.35 -> 60.7 mm
- net N$7: track 110.8 -> 57.8 mm, vias 1 -> 0
- net N$19: track 3.81 -> 56.2 mm
- net N$28: track 4.86 -> 55.0 mm
- net N$29: track 3.81 -> 47.6 mm, vias 0 -> 1
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